Commit message: Update Urdf_sandee_v1.urdf

File: URDF_sandee_v1/urdf/Urdf_sandee_v1.urdf (robot description, URDF)
Before this commit: robot Urdf_sandee_v1, 4 links, 3 joints
Joints:
- joint L_Wheel: limit lower=0 upper=0 effort=0 velocity=0 -> lower=-3.14 upper=3.14 effort=100.0 velocity=100.0
- joint R_Wheel: limit lower=0 upper=0 effort=0 velocity=0 -> lower=-3.14 upper=3.14 effort=100.0 velocity=100.0
